File: Swadge-HW/Swadge-2027-3V3.kicad_sch (KiCad schematic)
At the start: 8 parts, among them U10 M3410

Commit message: Annotations
Updated Annotations with zonal numbering
Parts:
- renumbered U10 to U5
Connections:
- net 3.3V renamed 3.3V_OUT
Changed lines of the file:
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@@
 		)
 	)
-	(label "3.3V"
+	(label "3.3V_OUT"
 		(at 162.56 63.5 0)
 		(effects
@@
 		)
 	)
-	(hierarchical_label "3.3V"
+	(hierarchical_label "3.3V_OUT"
 		(shape output)
 		(at 203.2 63.5 0)
@@
 		(in_pos_files yes)
 		(dnp no)
-		(property "Reference" "U10"
+		(property "Reference" "U5"
 			(at 130.81 72.644 0)
 			(show_name no)
@@
 			(project "Swadge-HW"
 				(path "/770c762f-3a30-4864-b7da-de353459cdd6/83e4033f-0c15-4157-a463-52f03cd15801/7daa4ba5-96fd-461d-be98-18bf8494bf52"
-					(reference "U10")
+					(reference "U5")
 					(unit 1)
 				)

Commit message: Starting PCB
Very Rough Initial Layout
Parts:
- renumbered C10 to C51, C12 to C52, C13 to C53, L4 to L51, R8 to R51, R18 to R52, R33 to R53
Changed lines of the file:
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@@
 		(in_pos_files yes)
 		(dnp no)
-		(property "Reference" "R18"
+		(property "Reference" "R52"
 			(at 176.784 80.0099 0)
 			(show_name no)
@@
 			(project "Swadge-HW"
 				(path "/770c762f-3a30-4864-b7da-de353459cdd6/83e4033f-0c15-4157-a463-52f03cd15801/7daa4ba5-96fd-461d-be98-18bf8494bf52"
-					(reference "R18")
+					(reference "R52")
 					(unit 1)
 				)
@@
 		(in_pos_files yes)
 		(dnp no)
-		(property "Reference" "R33"
+		(property "Reference" "R53"
 			(at 176.784 95.2499 0)
 			(show_name no)
@@
 			(project "Swadge-HW"
 				(path "/770c762f-3a30-4864-b7da-de353459cdd6/83e4033f-0c15-4157-a463-52f03cd15801/7daa4ba5-96fd-461d-be98-18bf8494bf52"
-					(reference "R33")
+					(reference "R53")
 					(unit 1)
 				)
@@
 		(in_pos_files yes)
 		(dnp no)
-		(property "Reference" "L4"
+		(property "Reference" "L51"
 			(at 153.67 59.69 90)
 			(show_name no)
@@
 			(project "Swadge-HW"
 				(path "/770c762f-3a30-4864-b7da-de353459cdd6/83e4033f-0c15-4157-a463-52f03cd15801/7daa4ba5-96fd-461d-be98-18bf8494bf52"
-					(reference "L4")
+					(reference "L51")
 					(unit 1)
 				)
@@
 		(in_pos_files yes)
 		(dnp no)
-		(property "Reference" "R8"
+		(property "Reference" "R51"
 			(at 176.784 69.8499 0)
 			(show_name no)
@@
 			(project "Swadge-HW"
 				(path "/770c762f-3a30-4864-b7da-de353459cdd6/83e4033f-0c15-4157-a463-52f03cd15801/7daa4ba5-96fd-461d-be98-18bf8494bf52"
-					(reference "R8")
+					(reference "R51")
 					(unit 1)
 				)
@@
 		(in_pos_files yes)
 		(dnp no)
-		(property "Reference" "C12"
+		(property "Reference" "C52"
 			(at 159.385 69.85 0)
 			(show_name no)
@@
 			(project "Swadge-HW"
 				(path "/770c762f-3a30-4864-b7da-de353459cdd6/83e4033f-0c15-4157-a463-52f03cd15801/7daa4ba5-96fd-461d-be98-18bf8494bf52"
-					(reference "C12")
+					(reference "C52")
 					(unit 1)
 				)
@@
 		(in_pos_files yes)
 		(dnp no)
-		(property "Reference" "C13"
+		(property "Reference" "C53"
 			(at 184.785 74.93 0)
 			(show_name no)
@@
 			(project "Swadge-HW"
 				(path "/770c762f-3a30-4864-b7da-de353459cdd6/83e4033f-0c15-4157-a463-52f03cd15801/7daa4ba5-96fd-461d-be98-18bf8494bf52"
-					(reference "C13")
+					(reference "C53")
 					(unit 1)
 				)
@@
 		(in_pos_files yes)
 		(dnp no)
-		(property "Reference" "C10"
+		(property "Reference" "C51"
 			(at 111.125 69.85 0)
 			(show_name no)
@@
 			(project "Swadge-HW"
 				(path "/770c762f-3a30-4864-b7da-de353459cdd6/83e4033f-0c15-4157-a463-52f03cd15801/7daa4ba5-96fd-461d-be98-18bf8494bf52"
-					(reference "C10")
+					(reference "C51")
 					(unit 1)
 				)

Commit message: major routing changes
Routed SPI
Started Test Routing Touch Inputs
Rough routing for LCD Power
Parts:
- C51, C52: Cost @ 2.5k (none) -> 0.0198; LCSC C59461 -> C159801
- C53: Cost @ 2.5k (none) -> 0.0066
- R51, R52: Cost @ 2.5k (none) -> 0.0022
- R53: Cost @ 2.5k (none) -> 0.0037
Changed lines of the file:
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@@
+			)
+		)
+		(property "Cost @ 2.5k" "0.0022"
+			(at 177.8 82.55 0)
+			(hide yes)
+			(show_name no)
+			(do_not_autoplace no)
+			(effects
+				(font
+					(size 1.27 1.27)
+				)
 			)
 		)
@@
 			)
 		)
+		(property "Cost @ 2.5k" "0.0037"
+			(at 177.8 97.79 0)
+			(hide yes)
+			(show_name no)
+			(do_not_autoplace no)
+			(effects
+				(font
+					(size 1.27 1.27)
+				)
+			)
+		)
 		(pin "1"
 		)
@@
 			)
 		)
+		(property "Cost @ 2.5k" "0.0022"
+			(at 177.8 72.39 0)
+			(hide yes)
+			(show_name no)
+			(do_not_autoplace no)
+			(effects
+				(font
+					(size 1.27 1.27)
+				)
+			)
+		)
 		(pin "1"
 		)
@@
 			)
 		)
-		(property "LCSC" "C59461"
+		(property "LCSC" "C159801"
+			(at 160.02 72.39 0)
+			(hide yes)
+			(show_name no)
+			(do_not_autoplace no)
+			(effects
+				(font
+					(size 1.27 1.27)
+				)
+			)
+		)
+		(property "Cost @ 2.5k" "0.0198"
 			(at 160.02 72.39 0)
 			(hide yes)
@@
 			)
 		)
+		(property "Cost @ 2.5k" "0.0066"
+			(at 185.42 77.47 0)
+			(hide yes)
+			(show_name no)
+			(do_not_autoplace no)
+			(effects
+				(font
+					(size 1.27 1.27)
+				)
+			)
+		)
 		(pin "2"
 		)
@@
 			)
 		)
-		(property "LCSC" "C59461"
+		(property "LCSC" "C159801"
 			(at 111.76 72.39 0)
 			(hide yes)
+			(show_name no)
+			(do_not_autoplace no)
+			(effects
+				(font
+					(size 1.27 1.27)
+				)
+			)
+		)
+		(property "Cost @ 2.5k" "0.0198"
+			(at 111.76 72.39 0)
+			(hide yes)
