File: Swadge-HW/Swadge-2027-ACC.kicad_sch (KiCad schematic)
At the start: 5 parts, among them U13 LSM6DSL

Commit message: Bus Renames
Since we really don't have that many signals I just ditched the bus prefixes and Alias'd them directly.
Added a bus for the interupt and status signals even if they are never used.
Connections:
- net ACC_INT1 renamed IMU_INT1
- net ACC_INT2 renamed IMU_INT2
- net COMM.I2C_SCL renamed I2C_SCL
- net COMM.I2C_SDA renamed I2C_SDA
Changed lines of the file:
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@@
+		)
+	)
+	(bus_entry
+		(at 93.98 96.52)
+		(size 2.54 2.54)
+		(stroke
+			(width 0)
+			(type default)
+		)
+	)
+	(bus_entry
+		(at 93.98 99.06)
+		(size 2.54 2.54)
+		(stroke
+			(width 0)
+			(type default)
+		)
+	)
+	(bus
+		(pts
+			(xy 86.36 86.36) (xy 93.98 86.36)
+		)
+		(stroke
+			(width 0)
+			(type default)
 		)
 	)
@@
 	(wire
 		(pts
-			(xy 157.48 99.06) (xy 193.04 99.06)
-		)
-		(stroke
-			(width 0)
-			(type default)
-		)
-	)
-	(wire
-		(pts
-			(xy 111.76 101.6) (xy 137.16 101.6)
+			(xy 157.48 99.06) (xy 185.42 99.06)
+		)
+		(stroke
+			(width 0)
+			(type default)
+		)
+	)
+	(bus
+		(pts
+			(xy 93.98 86.36) (xy 93.98 99.06)
 		)
 		(stroke
@@
 	(wire
 		(pts
+			(xy 96.52 99.06) (xy 111.76 99.06)
+		)
+		(stroke
+			(width 0)
+			(type default)
+		)
+	)
+	(wire
+		(pts
 			(xy 134.62 99.06) (xy 134.62 124.46)
 		)
@@
 	(wire
 		(pts
+			(xy 96.52 101.6) (xy 137.16 101.6)
+		)
+		(stroke
+			(width 0)
+			(type default)
+		)
+	)
+	(wire
+		(pts
 			(xy 129.54 68.58) (xy 129.54 111.76)
 		)
@@
 		)
 	)
-	(label "COMM.I2C_SDA"
+	(label "I2C_SDA"
 		(at 111.76 81.28 0)
 		(effects
@@
 		)
 	)
-	(label "COMM.I2C_SCL"
+	(label "I2C_SCL"
 		(at 111.76 78.74 0)
 		(effects
@@
 		)
 	)
-	(label "ACC_INT2"
-		(at 193.04 99.06 180)
+	(label "IMU_INT2"
+		(at 111.76 99.06 180)
 		(effects
 			(font
@@
 		)
 	)
-	(label "ACC_INT1"
-		(at 111.76 101.6 0)
+	(label "IMU_INT2"
+		(at 185.42 99.06 180)
+		(effects
+			(font
+				(size 1.27 1.27)
+			)
+			(justify right bottom)
+		)
+	)
+	(label "IMU_INT1"
+		(at 96.52 101.6 0)
 		(effects
 			(font
@@
 			)
 			(justify left bottom)
+		)
+	)
+	(hierarchical_label "{INTERUPTS}"
+		(shape input)
+		(at 86.36 86.36 180)
+		(effects
+			(font
+				(size 1.27 1.27)
+			)
+			(justify right)
 		)
 	)
@@
 		)
 	)
-	(hierarchical_label "COMM{COMM_BUS}"
+	(hierarchical_label "{COMM}"
 		(shape bidirectional)
 		(at 104.14 76.2 180)

Commit message: Annotations
Updated Annotations with zonal numbering
Parts:
- renumbered C34 to C71, C36 to C72, C35 to C73, R32 to R71, U13 to U7
Changed lines of the file:
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@@
 		(in_pos_files yes)
 		(dnp no)
-		(property "Reference" "C35"
+		(property "Reference" "C73"
 			(at 165.735 115.57 0)
 			(show_name no)
@@
 			(project "Swadge-HW"
 				(path "/770c762f-3a30-4864-b7da-de353459cdd6/d7da8eb8-65c1-44ec-ae93-82b297ca3e45"
-					(reference "C35")
+					(reference "C73")
 					(unit 1)
 				)
@@
 		(in_pos_files yes)
 		(dnp no)
-		(property "Reference" "C34"
+		(property "Reference" "C71"
 			(at 142.367 118.11 0)
 			(show_name no)
@@
 			(project "Swadge-HW"
 				(path "/770c762f-3a30-4864-b7da-de353459cdd6/d7da8eb8-65c1-44ec-ae93-82b297ca3e45"
-					(reference "C34")
+					(reference "C71")
 					(unit 1)
 				)
@@
 		(in_pos_files yes)
 		(dnp no)
-		(property "Reference" "R32"
+		(property "Reference" "R71"
 			(at 161.29 66.04 90)
 			(show_name no)
@@
 			(project "Swadge-HW"
 				(path "/770c762f-3a30-4864-b7da-de353459cdd6/d7da8eb8-65c1-44ec-ae93-82b297ca3e45"
-					(reference "R32")
+					(reference "R71")
 					(unit 1)
 				)
@@
 		(in_pos_files yes)
 		(dnp no)
-		(property "Reference" "C36"
+		(property "Reference" "C72"
 			(at 173.355 115.57 0)
 			(show_name no)
@@
 			(project "Swadge-HW"
 				(path "/770c762f-3a30-4864-b7da-de353459cdd6/d7da8eb8-65c1-44ec-ae93-82b297ca3e45"
-					(reference "C36")
+					(reference "C72")
 					(unit 1)
 				)
@@
 		(in_pos_files yes)
 		(dnp no)
-		(property "Reference" "U13"
+		(property "Reference" "U7"
 			(at 152.5113 84.836 0)
 			(show_name no)
@@
 			(project "Swadge-HW"
 				(path "/770c762f-3a30-4864-b7da-de353459cdd6/d7da8eb8-65c1-44ec-ae93-82b297ca3e45"
-					(reference "U13")
-					(unit 1)
-				)
+					(reference "U7")
+					(unit 1)
+				)

Commit message: major routing changes
Routed SPI
Started Test Routing Touch Inputs
Rough routing for LCD Power
Parts:
- C71, C72: Cost @ 2.5k 0.0015 -> 0.0182
- C73: Cost @ 2.5k 0.0079 -> 0.0198; LCSC C59461 -> C159801
- R71: Cost @ 2.5k 0.0008 -> 0.0018
Changed lines of the file:
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@@
 			)
 		)
-		(property "LCSC" "C59461"
+		(property "LCSC" "C159801"
 			(at 165.1 118.11 0)
 			(hide yes)
@@
 			)
 		)
-		(property "Cost @ 2.5k" "0.0079"
+		(property "Cost @ 2.5k" "0.0198"
 			(at 165.1 118.11 0)
 			(hide yes)
@@
 			)
 		)
-		(property "Cost @ 2.5k" "0.0015"
+		(property "Cost @ 2.5k" "0.0182"
 			(at 144.78 118.11 0)
 			(hide yes)
@@
 			)
 		)
-		(property "Cost @ 2.5k" "0.0008"
+		(property "Cost @ 2.5k" "0.0018"
 			(at 161.29 68.58 0)
 			(hide yes)
@@
 			)
 		)
-		(property "Cost @ 2.5k" "0.0015"
-			(at 172.72 118.11 0)
-			(hide yes)
+		(property "Cost @ 2.5k" "0.0182"
+			(at 172.72 118.11 0)
+			(hide yes)
