File: Swadge-HW/Swadge-2027-Lighting.kicad_sch (KiCad schematic)
At the start: 13 parts

Commit message: Bus Renames
Since we really don't have that many signals I just ditched the bus prefixes and Alias'd them directly.
Added a bus for the interupt and status signals even if they are never used.
Connections:
- net COMM.LED renamed LED
Changed lines of the file:
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@@
 		)
 	)
-	(label "COMM.LED"
+	(label "LED"
 		(at 45.72 66.04 0)
 		(effects
@@
 		)
 	)
-	(hierarchical_label "COMM{LED}"
+	(hierarchical_label "{COMM}"
 		(shape input)
 		(at 40.64 63.5 180)

Commit message: Annotations
Updated Annotations with zonal numbering
Parts:
- renumbered C6 to C26, C7 to C27, C21 to C28, C26 to C29, R13 to R22
Changed lines of the file:
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@@
 		(in_pos_files yes)
 		(dnp no)
-		(property "Reference" "C26"
+		(property "Reference" "C?"
 			(at 239.395 54.61 0)
 			(show_name no)
@@
 			(project "Swadge-HW"
 				(path "/770c762f-3a30-4864-b7da-de353459cdd6/5af7a925-0b98-46b1-b555-6a075ee725f5"
-					(reference "C26")
+					(reference "C?")
 					(unit 1)
 				)
@@
 		(in_pos_files yes)
 		(dnp no)
-		(property "Reference" "C21"
+		(property "Reference" "C?"
 			(at 188.595 54.61 0)
 			(show_name no)
@@
 			(project "Swadge-HW"
 				(path "/770c762f-3a30-4864-b7da-de353459cdd6/5af7a925-0b98-46b1-b555-6a075ee725f5"
-					(reference "C21")
+					(reference "C?")
 					(unit 1)
 				)
@@
 		(in_pos_files yes)
 		(dnp no)
-		(property "Reference" "R13"
+		(property "Reference" "R?"
 			(at 58.42 63.5 90)
 			(show_name no)
@@
 			(project "Swadge-HW"
 				(path "/770c762f-3a30-4864-b7da-de353459cdd6/5af7a925-0b98-46b1-b555-6a075ee725f5"
-					(reference "R13")
+					(reference "R?")
 					(unit 1)
 				)
@@
 		(in_pos_files yes)
 		(dnp no)
-		(property "Reference" "C7"
+		(property "Reference" "C?"
 			(at 137.795 54.61 0)
 			(show_name no)
@@
 			(project "Swadge-HW"
 				(path "/770c762f-3a30-4864-b7da-de353459cdd6/5af7a925-0b98-46b1-b555-6a075ee725f5"
-					(reference "C7")
+					(reference "C?")
 					(unit 1)
 				)
@@
 		(in_pos_files yes)
 		(dnp no)
-		(property "Reference" "C6"
+		(property "Reference" "C?"
 			(at 86.995 54.61 0)
 			(show_name no)
@@
 			(project "Swadge-HW"
 				(path "/770c762f-3a30-4864-b7da-de353459cdd6/5af7a925-0b98-46b1-b555-6a075ee725f5"
-					(reference "C6")
-					(unit 1)
-				)
+					(reference "C?")
+					(unit 1)
+				)

Commit message: Starting PCB
Very Rough Initial Layout
Parts:
- renumbered C26 to C906, C27 to C907, C28 to C908, C29 to C909, R22 to R910
Changed lines of the file:
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@@
 		)
 	)
-	(hierarchical_label "{COMM}"
+	(hierarchical_label "{PERIPHERAL}"
 		(shape input)
 		(at 40.64 63.5 180)
@@
 		(in_pos_files yes)
 		(dnp no)
-		(property "Reference" "C?"
+		(property "Reference" "C909"
 			(at 239.395 54.61 0)
 			(show_name no)
@@
 			(project "Swadge-HW"
 				(path "/770c762f-3a30-4864-b7da-de353459cdd6/5af7a925-0b98-46b1-b555-6a075ee725f5"
-					(reference "C?")
+					(reference "C909")
 					(unit 1)
 				)
@@
 		(in_pos_files yes)
 		(dnp no)
-		(property "Reference" "C?"
+		(property "Reference" "C908"
 			(at 188.595 54.61 0)
 			(show_name no)
@@
 			(project "Swadge-HW"
 				(path "/770c762f-3a30-4864-b7da-de353459cdd6/5af7a925-0b98-46b1-b555-6a075ee725f5"
-					(reference "C?")
+					(reference "C908")
 					(unit 1)
 				)
@@
 		(in_pos_files yes)
 		(dnp no)
-		(property "Reference" "R?"
+		(property "Reference" "R910"
 			(at 58.42 63.5 90)
 			(show_name no)
@@
 			(project "Swadge-HW"
 				(path "/770c762f-3a30-4864-b7da-de353459cdd6/5af7a925-0b98-46b1-b555-6a075ee725f5"
-					(reference "R?")
+					(reference "R910")
 					(unit 1)
 				)
@@
 		(in_pos_files yes)
 		(dnp no)
-		(property "Reference" "C?"
+		(property "Reference" "C907"
 			(at 137.795 54.61 0)
 			(show_name no)
@@
 			(project "Swadge-HW"
 				(path "/770c762f-3a30-4864-b7da-de353459cdd6/5af7a925-0b98-46b1-b555-6a075ee725f5"
-					(reference "C?")
+					(reference "C907")
 					(unit 1)
 				)
@@
 		(in_pos_files yes)
 		(dnp no)
-		(property "Reference" "C?"
+		(property "Reference" "C906"
 			(at 86.995 54.61 0)
 			(show_name no)
@@
 			(project "Swadge-HW"
 				(path "/770c762f-3a30-4864-b7da-de353459cdd6/5af7a925-0b98-46b1-b555-6a075ee725f5"
-					(reference "C?")
-					(unit 1)
-				)
+					(reference "C906")
+					(unit 1)
+				)

Commit message: major routing changes
Routed SPI
Started Test Routing Touch Inputs
Rough routing for LCD Power
Parts:
- C906, C907, C908, C909: Cost @ 2.5k (none) -> 0.0121
- D11, D12, D14, D15, D16, D17, D18, D19: Cost @ 2.5k (none) -> 0.0502
- R910: Cost @ 2.5k (none) -> 0.0018
Changed lines of the file:
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@@
+			)
+		)
+		(property "Cost @ 2.5k" "0.0502"
+			(at 254 66.04 0)
+			(hide yes)
+			(show_name no)
+			(do_not_autoplace no)
+			(effects
+				(font
+					(size 1.27 1.27)
+				)
 			)
 		)
@@
 			)
 		)
+		(property "Cost @ 2.5k" "0.0502"
+			(at 152.4 66.04 0)
+			(hide yes)
+			(show_name no)
+			(do_not_autoplace no)
+			(effects
+				(font
+					(size 1.27 1.27)
+				)
+			)
+		)
 		(pin "1"
 		)
@@
 			)
 		)
+		(property "Cost @ 2.5k" "0.0502"
+			(at 101.6 66.04 0)
+			(hide yes)
+			(show_name no)
+			(do_not_autoplace no)
+			(effects
+				(font
+					(size 1.27 1.27)
+				)
+			)
+		)
 		(pin "1"
 		)
@@
 				(font
 					(size 1 1)
+				)
+			)
+		)
+		(property "Cost @ 2.5k" "0.0502"
+			(at 177.8 66.04 0)
+			(hide yes)
+			(show_name no)
+			(do_not_autoplace no)
+			(effects
+				(font
+					(size 1.27 1.27)
 				)
 			)
@@
 			)
 		)
+		(property "Cost @ 2.5k" "0.0121"
+			(at 238.76 57.15 0)
+			(hide yes)
+			(show_name no)
+			(do_not_autoplace no)
+			(effects
+				(font
+					(size 1.27 1.27)
+				)
+			)
+		)
 		(pin "1"
 		)
@@
 				(font
 					(size 1 1)
+				)
+			)
+		)
+		(property "Cost @ 2.5k" "0.0502"
+			(at 203.2 66.04 0)
+			(hide yes)
+			(show_name no)
+			(do_not_autoplace no)
+			(effects
+				(font
+					(size 1.27 1.27)
 				)
 			)
@@
 		)
 		(property "LCSC" "C29936"
+			(at 187.96 57.15 0)
+			(hide yes)
+			(show_name no)
+			(do_not_autoplace no)
+			(effects
+				(font
+					(size 1.27 1.27)
+				)
+			)
+		)
+		(property "Cost @ 2.5k" "0.0121"
 			(at 187.96 57.15 0)
 			(hide yes)
@@
 			)
 		)
+		(property "Cost @ 2.5k" "0.0018"
+			(at 59.69 66.04 90)
+			(hide yes)
+			(show_name no)
+			(do_not_autoplace no)
+			(effects
+				(font
+					(size 1.27 1.27)
+				)
+			)
+		)
 		(pin "1"
 		)
@@
 			)
 		)
+		(property "Cost @ 2.5k" "0.0502"
+			(at 76.2 66.04 0)
+			(hide yes)
+			(show_name no)
+			(do_not_autoplace no)
+			(effects
+				(font
+					(size 1.27 1.27)
+				)
+			)
+		)
 		(pin "1"
 		)
@@
 				(font
 					(size 1 1)
+				)
+			)
+		)
+		(property "Cost @ 2.5k" "0.0502"
+			(at 228.6 66.04 0)
+			(hide yes)
+			(show_name no)
+			(do_not_autoplace no)
+			(effects
+				(font
+					(size 1.27 1.27)
 				)
 			)
@@
 			)
 		)
+		(property "Cost @ 2.5k" "0.0121"
+			(at 137.16 57.15 0)
+			(hide yes)
+			(show_name no)
+			(do_not_autoplace no)
+			(effects
+				(font
+					(size 1.27 1.27)
+				)
+			)
+		)
 		(pin "1"
 		)
@@
 			)
 		)
+		(property "Cost @ 2.5k" "0.0121"
+			(at 86.36 57.15 0)
+			(hide yes)
+			(show_name no)
+			(do_not_autoplace no)
+			(effects
+				(font
+					(size 1.27 1.27)
+				)
+			)
+		)
 		(pin "1"
 		)
@@
 				)
 			)
+		)
+		(property "Cost @ 2.5k" "0.0502"
+			(at 127 66.04 0)
+			(hide yes)
+			(show_name no)
+			(do_not_autoplace no)
+			(effects
+				(font
+					(size 1.27 1.27)
+				)
+			)
