File: Swadge-HW/Swadge-2027-RTC.kicad_sch (KiCad schematic)
At the start: 5 parts, among them U3 PCF8563DRG, Y1 32.768 kHz

Commit message: Annotations
Updated Annotations with zonal numbering
Parts:
- renumbered C17 to C61, C1 to C62, U3 to U6
Changed lines of the file:
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@@
 		(in_pos_files yes)
 		(dnp no)
-		(property "Reference" "C17"
+		(property "Reference" "C61"
 			(at 116.84 76.2 0)
 			(show_name no)
@@
 			(project "Swadge-HW"
 				(path "/770c762f-3a30-4864-b7da-de353459cdd6/54e099cb-7928-419d-b785-f2359f257eb1"
-					(reference "C17")
+					(reference "C61")
 					(unit 1)
 				)
@@
 		(dnp no)
 		(fields_autoplaced yes)
-		(property "Reference" "U3"
+		(property "Reference" "U6"
 			(at 146.9233 58.42 0)
 			(show_name no)
@@
 			(project "Swadge-HW"
 				(path "/770c762f-3a30-4864-b7da-de353459cdd6/54e099cb-7928-419d-b785-f2359f257eb1"
-					(reference "U3")
+					(reference "U6")
 					(unit 1)
 				)
@@
 		(in_pos_files yes)
 		(dnp no)
-		(property "Reference" "C1"
+		(property "Reference" "C62"
 			(at 104.14 76.2 0)
 			(show_name no)
@@
 			(project "Swadge-HW"
 				(path "/770c762f-3a30-4864-b7da-de353459cdd6/54e099cb-7928-419d-b785-f2359f257eb1"
-					(reference "C1")
+					(reference "C62")
 					(unit 1)
 				)

Commit message: major routing changes
Routed SPI
Started Test Routing Touch Inputs
Rough routing for LCD Power
Parts:
- C62: Substitutable (none) -> Y
- U6: Cost @ 2.5k (none) -> 0.0771
- Y1: Cost @ 2.5k (none) -> 0.0837
Changed lines of the file:
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@@
+			)
+		)
+		(property "Cost @ 2.5k" "0.0837"
+			(at 127 72.39 90)
+			(hide yes)
+			(show_name no)
+			(do_not_autoplace no)
+			(effects
+				(font
+					(size 1.27 1.27)
+				)
 			)
 		)
@@
 			)
 		)
+		(property "Cost @ 2.5k" "0.0771"
+			(at 144.78 71.12 0)
+			(hide yes)
+			(show_name no)
+			(do_not_autoplace no)
+			(effects
+				(font
+					(size 1.27 1.27)
+				)
+			)
+		)
 		(pin "7"
 		)
@@
 			(at 101.6 72.39 0)
 			(hide yes)
+			(show_name no)
+			(do_not_autoplace no)
+			(effects
+				(font
+					(size 1.27 1.27)
+				)
+			)
+		)
+		(property "Substitutable" "Y"
+			(at 101.6 72.39 0)
+			(hide yes)
