File: Swadge-HW/Swadge-2027-USB.kicad_sch (KiCad schematic)
At the start: 6 parts, among them P2 USB_C_Plug_USB2.0

Commit message: Bus Renames
Since we really don't have that many signals I just ditched the bus prefixes and Alias'd them directly.
Added a bus for the interupt and status signals even if they are never used.
Connections:
- net COMM.USB_D+ renamed USB_D+
- net COMM.USB_D- renamed USB_D-
Changed lines of the file:
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@@
 		)
 	)
-	(label "COMM.USB_D+"
+	(label "USB_D+"
 		(at 179.07 73.66 180)
 		(effects
@@
 		)
 	)
-	(label "COMM.USB_D-"
+	(label "USB_D-"
 		(at 179.07 81.28 180)
 		(effects
@@
 		)
 	)
-	(hierarchical_label "COMM{COMM_BUS}"
+	(hierarchical_label "{COMM}"
 		(shape bidirectional)
 		(at 195.58 86.36 0)

Commit message: Annotations
Updated Annotations with zonal numbering
Parts:
- renumbered P2 to P1
Connections:
- net EXT.USB_D+ renamed EXT_USB_D+
- net EXT.USB_D- renamed EXT_USB_D-
Changed lines of the file:
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@@
 		)
 	)
-	(label "EXT.USB_D-"
+	(label "EXT_USB_D-"
 		(at 129.54 78.74 180)
 		(effects
@@
 		)
 	)
-	(label "EXT.USB_D+"
+	(label "EXT_USB_D+"
 		(at 129.54 76.2 180)
 		(effects
@@
 		(in_pos_files yes)
 		(dnp no)
-		(property "Reference" "P2"
+		(property "Reference" "P1"
 			(at 86.36 59.69 0)
 			(show_name no)
@@
 			(project "Swadge-HW"
 				(path "/770c762f-3a30-4864-b7da-de353459cdd6/9586bcca-c960-42fc-9963-50259dda15b0"
-					(reference "P2")
-					(unit 1)
-				)
+					(reference "P1")
+					(unit 1)
+				)

Commit message: Cleanup
Renamed some components
Added in some net directives
Parts:
- renumbered D13 to D2, R30 to R19, R29 to R20, R23 to R21, R31 to R27
Changed lines of the file:
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@@
+		)
+	)
+	(rule_area
+		(exclude_from_sim no)
+		(in_bom yes)
+		(on_board yes)
+		(dnp no)
+		(polyline
+			(pts
+				(xy 163.83 71.12) (xy 163.83 83.82) (xy 166.37 83.82) (xy 166.37 71.12)
+			)
+			(stroke
+				(width 0)
+				(type dash)
+			)
+			(fill
+				(type none)
+			)
+		)
+	)
+	(rule_area
+		(exclude_from_sim no)
+		(in_bom yes)
+		(on_board yes)
+		(dnp no)
+		(polyline
+			(pts
+				(xy 135.8588 73.66) (xy 135.8588 81.28) (xy 138.3988 81.28) (xy 138.3988 73.66)
+			)
+			(stroke
+				(width 0)
+				(type dash)
+			)
+			(fill
+				(type none)
+			)
+		)
+	)
+	(netclass_flag ""
+		(length 2.54)
+		(shape round)
+		(at 165.1 71.12 0)
+		(fields_autoplaced yes)
+		(effects
+			(font
+				(size 1.27 1.27)
+			)
+			(justify left bottom)
+		)
+		(property "Netclass" "Comm_TP"
+			(at 165.7985 68.58 0)
+			(show_name no)
+			(do_not_autoplace no)
+			(effects
+				(font
+					(size 1.27 1.27)
+				)
+				(justify left)
+			)
+		)
+		(property "Component Class" ""
+			(at -167.64 40.64 0)
+			(show_name no)
+			(do_not_autoplace no)
+			(effects
+				(font
+					(size 1.27 1.27)
+					(italic yes)
+				)
+			)
+		)
+	)
+	(netclass_flag ""
+		(length 2.54)
+		(shape round)
+		(at 137.1288 73.66 0)
+		(fields_autoplaced yes)
+		(effects
+			(font
+				(size 1.27 1.27)
+			)
+			(justify left bottom)
+		)
+		(property "Netclass" "Comm_TP"
+			(at 137.8273 71.12 0)
+			(show_name no)
+			(do_not_autoplace no)
+			(effects
+				(font
+					(size 1.27 1.27)
+				)
+				(justify left)
+			)
+		)
+		(property "Component Class" ""
+			(at -195.6112 43.18 0)
+			(show_name no)
+			(do_not_autoplace no)
+			(effects
+				(font
+					(size 1.27 1.27)
+					(italic yes)
+				)
+			)
 		)
 	)
@@
 		(in_pos_files yes)
 		(dnp no)
-		(property "Reference" "R31"
+		(property "Reference" "R?"
 			(at 154.94 102.87 90)
 			(show_name no)
@@
 			(project "Swadge-HW"
 				(path "/770c762f-3a30-4864-b7da-de353459cdd6/9586bcca-c960-42fc-9963-50259dda15b0"
-					(reference "R31")
+					(reference "R?")
 					(unit 1)
 				)
@@
 		(in_pos_files yes)
 		(dnp no)
-		(property "Reference" "R30"
+		(property "Reference" "R?"
 			(at 150.114 79.248 90)
 			(show_name no)
@@
 			(project "Swadge-HW"
 				(path "/770c762f-3a30-4864-b7da-de353459cdd6/9586bcca-c960-42fc-9963-50259dda15b0"
-					(reference "R30")
+					(reference "R?")
 					(unit 1)
 				)
@@
 		(in_pos_files yes)
 		(dnp no)
-		(property "Reference" "R23"
+		(property "Reference" "R?"
 			(at 144.78 102.87 90)
 			(show_name no)
@@
 			(project "Swadge-HW"
 				(path "/770c762f-3a30-4864-b7da-de353459cdd6/9586bcca-c960-42fc-9963-50259dda15b0"
-					(reference "R23")
+					(reference "R?")
 					(unit 1)
 				)
@@
 		(in_pos_files yes)
 		(dnp no)
-		(property "Reference" "R29"
+		(property "Reference" "R?"
 			(at 151.13 71.374 90)
 			(show_name no)
@@
 			(project "Swadge-HW"
 				(path "/770c762f-3a30-4864-b7da-de353459cdd6/9586bcca-c960-42fc-9963-50259dda15b0"
-					(reference "R29")
+					(reference "R?")
 					(unit 1)
 				)
@@
 		(in_pos_files yes)
 		(dnp no)
-		(property "Reference" "D13"
+		(property "Reference" "D?"
 			(at 127 109.22 0)
 			(show_name no)
@@
 			(project "Swadge-HW"
 				(path "/770c762f-3a30-4864-b7da-de353459cdd6/9586bcca-c960-42fc-9963-50259dda15b0"
-					(reference "D13")
-					(unit 1)
-				)
+					(reference "D?")
+					(unit 1)
+				)

Commit message: Starting PCB
Very Rough Initial Layout
Parts:
- renumbered D2 to D901, R21 to R906, R20 to R907, R19 to R908, R27 to R909
Changed lines of the file:
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@@
 		(in_pos_files yes)
 		(dnp no)
-		(property "Reference" "R?"
+		(property "Reference" "R909"
 			(at 154.94 102.87 90)
 			(show_name no)
@@
 			(project "Swadge-HW"
 				(path "/770c762f-3a30-4864-b7da-de353459cdd6/9586bcca-c960-42fc-9963-50259dda15b0"
-					(reference "R?")
+					(reference "R909")
 					(unit 1)
 				)
@@
 		(in_pos_files yes)
 		(dnp no)
-		(property "Reference" "R?"
+		(property "Reference" "R908"
 			(at 150.114 79.248 90)
 			(show_name no)
@@
 			(project "Swadge-HW"
 				(path "/770c762f-3a30-4864-b7da-de353459cdd6/9586bcca-c960-42fc-9963-50259dda15b0"
-					(reference "R?")
+					(reference "R908")
 					(unit 1)
 				)
@@
 		(in_pos_files yes)
 		(dnp no)
-		(property "Reference" "R?"
+		(property "Reference" "R906"
 			(at 144.78 102.87 90)
 			(show_name no)
@@
 			(project "Swadge-HW"
 				(path "/770c762f-3a30-4864-b7da-de353459cdd6/9586bcca-c960-42fc-9963-50259dda15b0"
-					(reference "R?")
+					(reference "R906")
 					(unit 1)
 				)
@@
 		(in_pos_files yes)
 		(dnp no)
-		(property "Reference" "R?"
+		(property "Reference" "R907"
 			(at 151.13 71.374 90)
 			(show_name no)
@@
 			(project "Swadge-HW"
 				(path "/770c762f-3a30-4864-b7da-de353459cdd6/9586bcca-c960-42fc-9963-50259dda15b0"
-					(reference "R?")
+					(reference "R907")
 					(unit 1)
 				)
@@
 		(in_pos_files yes)
 		(dnp no)
-		(property "Reference" "D?"
+		(property "Reference" "D901"
 			(at 127 109.22 0)
 			(show_name no)
@@
 			(project "Swadge-HW"
 				(path "/770c762f-3a30-4864-b7da-de353459cdd6/9586bcca-c960-42fc-9963-50259dda15b0"
-					(reference "D?")
-					(unit 1)
-				)
+					(reference "D901")
+					(unit 1)
+				)

Commit message: major routing changes
Routed SPI
Started Test Routing Touch Inputs
Rough routing for LCD Power
Parts:
- R906, R909: Cost @ 2.5k (none) -> 0.0023
- R907, R908: Cost @ 2.5k (none) -> 0.0018
Changed lines of the file:
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@@
+			)
+		)
+		(property "Cost @ 2.5k" "0.0023"
+			(at 157.48 102.87 90)
+			(hide yes)
+			(show_name no)
+			(do_not_autoplace no)
+			(effects
+				(font
+					(size 1.27 1.27)
+				)
 			)
 		)
@@
 			)
 		)
+		(property "Cost @ 2.5k" "0.0018"
+			(at 153.67 81.28 90)
+			(hide yes)
+			(show_name no)
+			(do_not_autoplace no)
+			(effects
+				(font
+					(size 1.27 1.27)
+				)
+			)
+		)
 		(pin "1"
 		)
@@
 		)
 		(property "LCSC" "C2907044"
+			(at 147.32 102.87 90)
+			(hide yes)
+			(show_name no)
+			(do_not_autoplace no)
+			(effects
+				(font
+					(size 1.27 1.27)
+				)
+			)
+		)
+		(property "Cost @ 2.5k" "0.0023"
 			(at 147.32 102.87 90)
 			(hide yes)
@@
 			(at 153.67 73.66 90)
 			(hide yes)
+			(show_name no)
+			(do_not_autoplace no)
+			(effects
+				(font
+					(size 1.27 1.27)
+				)
+			)
+		)
+		(property "Cost @ 2.5k" "0.0018"
+			(at 153.67 73.66 90)
+			(hide yes)
