File: Swadge-HW/Swadge-2027-IO.kicad_sch (KiCad schematic)
At the start: 22 parts, among them SW10 B3FS-4002P, SW11 B3FS-4002P, SW12 YTS-D003-1A, SW13 YTS-D003-1A, SW14 YTS-D003-1A, SW15 YTS-D003-1A, SW16 YTS-D003-1A, SW17 YTS-D003-1A

Commit message: Annotations
Updated Annotations with zonal numbering
Parts:
- renumbered U4 to S1, U14 to S2
Changed lines of the file:
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@@
 		(in_pos_files yes)
 		(dnp yes)
-		(property "Reference" "U14"
+		(property "Reference" "S2"
 			(at 217.17 81.28 0)
 			(show_name no)
@@
 			(project "Swadge-HW"
 				(path "/770c762f-3a30-4864-b7da-de353459cdd6/124674ec-3e27-486f-b028-a72f7ae9e19e"
-					(reference "U14")
+					(reference "S2")
 					(unit 1)
 				)
@@
 		(in_pos_files yes)
 		(dnp yes)
-		(property "Reference" "U4"
+		(property "Reference" "S1"
 			(at 217.17 38.1 0)
 			(show_name no)
@@
 			(project "Swadge-HW"
 				(path "/770c762f-3a30-4864-b7da-de353459cdd6/124674ec-3e27-486f-b028-a72f7ae9e19e"
-					(reference "U4")
+					(reference "S1")
 					(unit 1)
 				)

Commit message: Starting PCB
Very Rough Initial Layout
Parts:
- renumbered R10 to R101, R11 to R102, R12 to R103, R15 to R104, R16 to R105, R17 to R106, R14 to R107, R24 to R108, R25 to R109, R27 to R110, R28 to R111, R34 to R112
Changed lines of the file:
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@@
 		(in_pos_files yes)
 		(dnp no)
-		(property "Reference" "R17"
+		(property "Reference" "R106"
 			(at 239.014 53.34 90)
 			(show_name no)
@@
 			(project "Swadge-HW"
 				(path "/770c762f-3a30-4864-b7da-de353459cdd6/124674ec-3e27-486f-b028-a72f7ae9e19e"
-					(reference "R17")
+					(reference "R106")
 					(unit 1)
 				)
@@
 		(in_pos_files yes)
 		(dnp no)
-		(property "Reference" "R16"
+		(property "Reference" "R105"
 			(at 239.014 50.8 90)
 			(show_name no)
@@
 			(project "Swadge-HW"
 				(path "/770c762f-3a30-4864-b7da-de353459cdd6/124674ec-3e27-486f-b028-a72f7ae9e19e"
-					(reference "R16")
+					(reference "R105")
 					(unit 1)
 				)
@@
 		(in_pos_files yes)
 		(dnp no)
-		(property "Reference" "R15"
+		(property "Reference" "R104"
 			(at 239.014 48.26 90)
 			(show_name no)
@@
 			(project "Swadge-HW"
 				(path "/770c762f-3a30-4864-b7da-de353459cdd6/124674ec-3e27-486f-b028-a72f7ae9e19e"
-					(reference "R15")
+					(reference "R104")
 					(unit 1)
 				)
@@
 		(in_pos_files yes)
 		(dnp no)
-		(property "Reference" "R25"
+		(property "Reference" "R109"
 			(at 239.014 88.9 90)
 			(show_name no)
@@
 			(project "Swadge-HW"
 				(path "/770c762f-3a30-4864-b7da-de353459cdd6/124674ec-3e27-486f-b028-a72f7ae9e19e"
-					(reference "R25")
+					(reference "R109")
 					(unit 1)
 				)
@@
 		(in_pos_files yes)
 		(dnp no)
-		(property "Reference" "R12"
+		(property "Reference" "R103"
 			(at 239.014 45.72 90)
 			(show_name no)
@@
 			(project "Swadge-HW"
 				(path "/770c762f-3a30-4864-b7da-de353459cdd6/124674ec-3e27-486f-b028-a72f7ae9e19e"
-					(reference "R12")
+					(reference "R103")
 					(unit 1)
 				)
@@
 		(in_pos_files yes)
 		(dnp no)
-		(property "Reference" "R24"
+		(property "Reference" "R108"
 			(at 239.014 86.36 90)
 			(show_name no)
@@
 			(project "Swadge-HW"
 				(path "/770c762f-3a30-4864-b7da-de353459cdd6/124674ec-3e27-486f-b028-a72f7ae9e19e"
-					(reference "R24")
+					(reference "R108")
 					(unit 1)
 				)
@@
 		(in_pos_files yes)
 		(dnp no)
-		(property "Reference" "R34"
+		(property "Reference" "R112"
 			(at 239.014 96.52 90)
 			(show_name no)
@@
 			(project "Swadge-HW"
 				(path "/770c762f-3a30-4864-b7da-de353459cdd6/124674ec-3e27-486f-b028-a72f7ae9e19e"
-					(reference "R34")
+					(reference "R112")
 					(unit 1)
 				)
@@
 		(in_pos_files yes)
 		(dnp no)
-		(property "Reference" "R14"
+		(property "Reference" "R107"
 			(at 239.014 83.82 90)
 			(show_name no)
@@
 			(project "Swadge-HW"
 				(path "/770c762f-3a30-4864-b7da-de353459cdd6/124674ec-3e27-486f-b028-a72f7ae9e19e"
-					(reference "R14")
+					(reference "R107")
 					(unit 1)
 				)
@@
 		(in_pos_files yes)
 		(dnp no)
-		(property "Reference" "R11"
+		(property "Reference" "R102"
 			(at 239.014 43.18 90)
 			(show_name no)
@@
 			(project "Swadge-HW"
 				(path "/770c762f-3a30-4864-b7da-de353459cdd6/124674ec-3e27-486f-b028-a72f7ae9e19e"
-					(reference "R11")
+					(reference "R102")
 					(unit 1)
 				)
@@
 		(in_pos_files yes)
 		(dnp no)
-		(property "Reference" "R28"
+		(property "Reference" "R111"
 			(at 239.014 93.98 90)
 			(show_name no)
@@
 			(project "Swadge-HW"
 				(path "/770c762f-3a30-4864-b7da-de353459cdd6/124674ec-3e27-486f-b028-a72f7ae9e19e"
-					(reference "R28")
+					(reference "R111")
 					(unit 1)
 				)
@@
 		(in_pos_files yes)
 		(dnp no)
-		(property "Reference" "R10"
+		(property "Reference" "R101"
 			(at 239.014 40.64 90)
 			(show_name no)
@@
 			(project "Swadge-HW"
 				(path "/770c762f-3a30-4864-b7da-de353459cdd6/124674ec-3e27-486f-b028-a72f7ae9e19e"
-					(reference "R10")
+					(reference "R101")
 					(unit 1)
 				)
@@
 		(in_pos_files yes)
 		(dnp no)
-		(property "Reference" "R27"
+		(property "Reference" "R110"
 			(at 239.014 91.44 90)
 			(show_name no)
@@
 			(project "Swadge-HW"
 				(path "/770c762f-3a30-4864-b7da-de353459cdd6/124674ec-3e27-486f-b028-a72f7ae9e19e"
-					(reference "R27")
+					(reference "R110")
 					(unit 1)
 				)

Commit message: major routing changes
Routed SPI
Started Test Routing Touch Inputs
Rough routing for LCD Power
Parts:
- SW10, SW11: Cost @ 2.5k (none) -> 0.0598
Changed lines of the file:
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@@
+			)
+		)
+		(property "Cost @ 2.5k" "0.0598"
+			(at 114.3 147.32 90)
+			(hide yes)
+			(show_name no)
+			(do_not_autoplace no)
+			(effects
+				(font
+					(size 1.27 1.27)
+				)
 			)
 		)
@@
 				)
 			)
+		)
+		(property "Cost @ 2.5k" "0.0598"
+			(at 114.3 167.64 90)
+			(hide yes)
+			(show_name no)
+			(do_not_autoplace no)
+			(effects
+				(font
+					(size 1.27 1.27)
+				)
+			)
