File: Swadge-HW/Swadge-2027-BMS.kicad_sch (KiCad schematic)
At the start: 10 parts, among them U12 BQ24259

Commit message: Annotations
Updated Annotations with zonal numbering
Parts:
- renumbered U12 to U4
Changed lines of the file:
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@@
+		)
+	)
+	(hierarchical_label "REGN"
+		(shape output)
+		(at 170.18 48.26 0)
+		(effects
+			(font
+				(size 1.27 1.27)
+			)
+			(justify left)
 		)
 	)
@@
 		(dnp no)
 		(fields_autoplaced yes)
-		(property "Reference" "U12"
+		(property "Reference" "U4"
 			(at 147.32 29.0025 0)
 			(show_name no)
@@
 			(project "Swadge-HW"
 				(path "/770c762f-3a30-4864-b7da-de353459cdd6/83e4033f-0c15-4157-a463-52f03cd15801/fcbd4cfc-9cd2-46ce-8965-013db5b57f46"
-					(reference "U12")
+					(reference "U4")
 					(unit 1)
 				)

Commit message: Starting PCB
Very Rough Initial Layout
Parts:
- C41: renamed from C28; footprint Capacitor_SMD:C_0603_1608Metric -> Swadge_Parts:C_0603_1608Metric
- renumbered C31 to C42, C32 to C43, C33 to C44, C27 to C45, C29 to C46, C30 to C47, L2 to L41, R20 to R41
Changed lines of the file:
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@@
 		(in_pos_files yes)
 		(dnp no)
-		(property "Reference" "C33"
+		(property "Reference" "C44"
 			(at 223.52 45.72 0)
 			(show_name no)
@@
 			(project "Swadge-HW"
 				(path "/770c762f-3a30-4864-b7da-de353459cdd6/83e4033f-0c15-4157-a463-52f03cd15801/fcbd4cfc-9cd2-46ce-8965-013db5b57f46"
-					(reference "C33")
+					(reference "C44")
 					(unit 1)
 				)
@@
 		(in_pos_files yes)
 		(dnp no)
-		(property "Reference" "C32"
+		(property "Reference" "C43"
 			(at 208.28 45.72 0)
 			(show_name no)
@@
 			(project "Swadge-HW"
 				(path "/770c762f-3a30-4864-b7da-de353459cdd6/83e4033f-0c15-4157-a463-52f03cd15801/fcbd4cfc-9cd2-46ce-8965-013db5b57f46"
-					(reference "C32")
+					(reference "C43")
 					(unit 1)
 				)
@@
 		(in_pos_files yes)
 		(dnp no)
-		(property "Reference" "C31"
+		(property "Reference" "C42"
 			(at 180.34 71.12 0)
 			(show_name no)
@@
 			(project "Swadge-HW"
 				(path "/770c762f-3a30-4864-b7da-de353459cdd6/83e4033f-0c15-4157-a463-52f03cd15801/fcbd4cfc-9cd2-46ce-8965-013db5b57f46"
-					(reference "C31")
+					(reference "C42")
 					(unit 1)
 				)
@@
 		(in_pos_files yes)
 		(dnp no)
-		(property "Reference" "C27"
+		(property "Reference" "C45"
 			(at 53.34 90.17 0)
 			(show_name no)
@@
 			(project "Swadge-HW"
 				(path "/770c762f-3a30-4864-b7da-de353459cdd6/83e4033f-0c15-4157-a463-52f03cd15801/fcbd4cfc-9cd2-46ce-8965-013db5b57f46"
-					(reference "C27")
+					(reference "C45")
 					(unit 1)
 				)
@@
 		(in_pos_files yes)
 		(dnp no)
-		(property "Reference" "R20"
+		(property "Reference" "R41"
 			(at 103.632 53.848 0)
 			(show_name no)
@@
 			(project "Swadge-HW"
 				(path "/770c762f-3a30-4864-b7da-de353459cdd6/83e4033f-0c15-4157-a463-52f03cd15801/fcbd4cfc-9cd2-46ce-8965-013db5b57f46"
-					(reference "R20")
+					(reference "R41")
 					(unit 1)
 				)
@@
 		(in_pos_files yes)
 		(dnp no)
-		(property "Reference" "C29"
+		(property "Reference" "C46"
 			(at 96.52 90.17 0)
 			(show_name no)
@@
 			(project "Swadge-HW"
 				(path "/770c762f-3a30-4864-b7da-de353459cdd6/83e4033f-0c15-4157-a463-52f03cd15801/fcbd4cfc-9cd2-46ce-8965-013db5b57f46"
-					(reference "C29")
+					(reference "C46")
 					(unit 1)
 				)
@@
 		(dnp no)
 		(fields_autoplaced yes)
-		(property "Reference" "C28"
+		(property "Reference" "C41"
 			(at 90.17 40.6399 0)
 			(show_name no)
@@
 			)
 		)
-		(property "Footprint" "Capacitor_SMD:C_0603_1608Metric"
+		(property "Footprint" "Swadge_Parts:C_0603_1608Metric"
 			(at 87.3252 45.72 0)
 			(hide yes)
@@
 			(project "Swadge-HW"
 				(path "/770c762f-3a30-4864-b7da-de353459cdd6/83e4033f-0c15-4157-a463-52f03cd15801/fcbd4cfc-9cd2-46ce-8965-013db5b57f46"
-					(reference "C28")
+					(reference "C41")
 					(unit 1)
 				)
@@
 		(in_pos_files yes)
 		(dnp no)
-		(property "Reference" "L2"
+		(property "Reference" "L41"
 			(at 179.07 34.29 90)
 			(show_name no)
@@
 			(project "Swadge-HW"
 				(path "/770c762f-3a30-4864-b7da-de353459cdd6/83e4033f-0c15-4157-a463-52f03cd15801/fcbd4cfc-9cd2-46ce-8965-013db5b57f46"
-					(reference "L2")
+					(reference "L41")
 					(unit 1)
 				)
@@
 		(in_pos_files yes)
 		(dnp no)
-		(property "Reference" "C30"
+		(property "Reference" "C47"
 			(at 109.22 90.17 0)
 			(show_name no)
@@
 			(project "Swadge-HW"
 				(path "/770c762f-3a30-4864-b7da-de353459cdd6/83e4033f-0c15-4157-a463-52f03cd15801/fcbd4cfc-9cd2-46ce-8965-013db5b57f46"
-					(reference "C30")
+					(reference "C47")
 					(unit 1)
 				)

Commit message: major routing changes
Routed SPI
Started Test Routing Touch Inputs
Rough routing for LCD Power
Parts:
- C41: Cost @ 2.5k 0.0079 -> 0.0121; LCSC C159801 -> C29936
- C45: Cost @ 2.5k (none) -> 0.0071
- C46: Cost @ 2.5k (none) -> 0.0109
- C47: Cost @ 2.5k (none) -> 0.0576
Changed lines of the file:
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@@
+			)
+		)
+		(property "Cost @ 2.5k" "0.0071"
+			(at 55.88 87.63 0)
+			(hide yes)
+			(show_name no)
+			(do_not_autoplace no)
+			(effects
+				(font
+					(size 1.27 1.27)
+				)
 			)
 		)
@@
 			)
 		)
+		(property "Cost @ 2.5k" "0.0109"
+			(at 99.06 87.63 0)
+			(hide yes)
+			(show_name no)
+			(do_not_autoplace no)
+			(effects
+				(font
+					(size 1.27 1.27)
+				)
+			)
+		)
 		(pin "1"
 		)
@@
 			)
 		)
-		(property "LCSC" "C159801"
+		(property "LCSC" "C29936"
 			(at 86.36 41.91 0)
 			(hide yes)
@@
 			)
 		)
-		(property "Cost @ 2.5k" "0.0079"
+		(property "Cost @ 2.5k" "0.0121"
 			(at 86.36 41.91 0)
 			(hide yes)
@@
 			(at 111.76 87.63 0)
 			(hide yes)
+			(show_name no)
+			(do_not_autoplace no)
+			(effects
+				(font
+					(size 1.27 1.27)
+				)
+			)
+		)
+		(property "Cost @ 2.5k" "0.0576"
+			(at 111.76 87.63 0)
+			(hide yes)

Commit message: Layout Changes
Moved USB 10deg around perimeter to get it closer to the ESP32 and the left thigh.
Substantially compressed BMS and 3.3V layout
Started Routing the Touch Inputs
Other:
- note added: "BQ24259 Switches at 1.5Mhz Default Vsys_min set at 3.5V Vsys = Vbatt when Vbatt > Vsys_min"
- note removed: "BQ24259 Switches at 1.2Mhz"
Changed lines of the file:
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@@
 		)
 	)
-	(text "BQ24259 Switches at 1.2Mhz"
+	(text "BQ24259 Switches at 1.5Mhz\nDefault Vsys_min set at 3.5V\nVsys = Vbatt when Vbatt > Vsys_min"
 		(exclude_from_sim no)
 		(at 134.62 25.4 0)
