File: Swadge-HW/Swadge-2027-LCD.kicad_sch (KiCad schematic)
At the start: 14 parts, among them Q1 Q_PMOS_GSD, U2 RB017A1505A, U5 RB017A1505A_Connector, U7 GENERIC_LDO_GOI

Commit message: Bus Renames
Since we really don't have that many signals I just ditched the bus prefixes and Alias'd them directly.
Added a bus for the interupt and status signals even if they are never used.
Connections:
- net COMM.FSPI_CS0 renamed FSPI_CS0
- net PERF.TFT_ATP renamed TFT_ATP
- net PERF.TFT_RESET renamed TFT_RESET
- net PERF.TFT_RS renamed TFT_RS
Changed lines of the file:
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@@
 		)
 	)
-	(label "PERF.TFT_ATP"
+	(label "TFT_ATP"
 		(at 154.94 93.98 180)
 		(effects
@@
 		)
 	)
-	(label "PERF.TFT_RS"
+	(label "TFT_RS"
 		(at 160.02 101.6 0)
 		(effects
@@
 		)
 	)
-	(label "PERF.TFT_RESET"
+	(label "TFT_RESET"
 		(at 160.02 109.22 0)
 		(effects
@@
 		)
 	)
-	(label "COMM.FSPI_CS0"
+	(label "FSPI_CS0"
 		(at 187.96 86.36 0)
 		(effects
@@
 		)
 	)
-	(hierarchical_label "COMM{COMM_BUS}"
+	(hierarchical_label "{COMM}"
 		(shape bidirectional)
 		(at 180.34 78.74 180)
@@
 		)
 	)
-	(hierarchical_label "PERF{PERF_BUS}"
+	(hierarchical_label "{PERIPHERAL}"
 		(shape input)
 		(at 152.4 83.82 180)

Commit message: Annotations
Updated Annotations with zonal numbering
Parts:
- renumbered C16 to C91, C19 to C92, C23 to C93, C25 to C94, C11 to C95, C22 to C96, U2 to DS1, U5 to P2, R7 to R91, R26 to R92, U7 to U9
Changed lines of the file:
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@@
 		(in_pos_files yes)
 		(dnp no)
-		(property "Reference" "U2"
+		(property "Reference" "DS1"
 			(at 218.44 86.36 0)
 			(show_name no)
@@
 			(project "Swadge-HW"
 				(path "/770c762f-3a30-4864-b7da-de353459cdd6/50e190c4-5ab4-41d8-900d-31bbecb31a92"
-					(reference "U2")
+					(reference "DS1")
 					(unit 1)
 				)
@@
 		(in_pos_files yes)
 		(dnp no)
-		(property "Reference" "U5"
+		(property "Reference" "P2"
 			(at 219.71 67.31 0)
 			(show_name no)
@@
 			(project "Swadge-HW"
 				(path "/770c762f-3a30-4864-b7da-de353459cdd6/50e190c4-5ab4-41d8-900d-31bbecb31a92"
-					(reference "U5")
+					(reference "P2")
 					(unit 1)
 				)
@@
 		(in_pos_files yes)
 		(dnp no)
-		(property "Reference" "C23"
+		(property "Reference" "C93"
 			(at 239.395 105.41 0)
 			(show_name no)
@@
 			(project "Swadge-HW"
 				(path "/770c762f-3a30-4864-b7da-de353459cdd6/50e190c4-5ab4-41d8-900d-31bbecb31a92"
-					(reference "C23")
+					(reference "C93")
 					(unit 1)
 				)
@@
 		(in_pos_files yes)
 		(dnp no)
-		(property "Reference" "R26"
+		(property "Reference" "R92"
 			(at 180.34 124.46 90)
 			(show_name no)
@@
 			(project "Swadge-HW"
 				(path "/770c762f-3a30-4864-b7da-de353459cdd6/50e190c4-5ab4-41d8-900d-31bbecb31a92"
-					(reference "R26")
+					(reference "R92")
 					(unit 1)
 				)
@@
 		(in_pos_files yes)
 		(dnp no)
-		(property "Reference" "C11"
+		(property "Reference" "C95"
 			(at 79.375 118.11 0)
 			(show_name no)
@@
 			(project "Swadge-HW"
 				(path "/770c762f-3a30-4864-b7da-de353459cdd6/50e190c4-5ab4-41d8-900d-31bbecb31a92"
-					(reference "C11")
+					(reference "C95")
 					(unit 1)
 				)
@@
 		(in_pos_files yes)
 		(dnp no)
-		(property "Reference" "U7"
+		(property "Reference" "U9"
 			(at 99.06 45.72 0)
 			(show_name no)
@@
 			(project "Swadge-HW"
 				(path "/770c762f-3a30-4864-b7da-de353459cdd6/50e190c4-5ab4-41d8-900d-31bbecb31a92"
-					(reference "U7")
+					(reference "U9")
 					(unit 1)
 				)
@@
 		(in_pos_files yes)
 		(dnp no)
-		(property "Reference" "C25"
+		(property "Reference" "C94"
 			(at 247.015 105.41 0)
 			(show_name no)
@@
 			(project "Swadge-HW"
 				(path "/770c762f-3a30-4864-b7da-de353459cdd6/50e190c4-5ab4-41d8-900d-31bbecb31a92"
-					(reference "C25")
+					(reference "C94")
 					(unit 1)
 				)
@@
 		(in_pos_files yes)
 		(dnp no)
-		(property "Reference" "C19"
+		(property "Reference" "C92"
 			(at 119.253 41.91 0)
 			(show_name no)
@@
 			(project "Swadge-HW"
 				(path "/770c762f-3a30-4864-b7da-de353459cdd6/50e190c4-5ab4-41d8-900d-31bbecb31a92"
-					(reference "C19")
+					(reference "C92")
 					(unit 1)
 				)
@@
 		(in_pos_files yes)
 		(dnp no)
-		(property "Reference" "R7"
+		(property "Reference" "R91"
 			(at 83.82 102.87 90)
 			(show_name no)
@@
 			(project "Swadge-HW"
 				(path "/770c762f-3a30-4864-b7da-de353459cdd6/50e190c4-5ab4-41d8-900d-31bbecb31a92"
-					(reference "R7")
+					(reference "R91")
 					(unit 1)
 				)
@@
 		(dnp no)
 		(fields_autoplaced yes)
-		(property "Reference" "C22"
+		(property "Reference" "C96"
 			(at 123.19 119.3799 0)
 			(show_name no)
@@
 			(project "Swadge-HW"
 				(path "/770c762f-3a30-4864-b7da-de353459cdd6/50e190c4-5ab4-41d8-900d-31bbecb31a92"
-					(reference "C22")
+					(reference "C96")
 					(unit 1)
 				)
@@
 		(in_pos_files yes)
 		(dnp no)
-		(property "Reference" "C16"
+		(property "Reference" "C91"
 			(at 83.185 39.37 0)
 			(show_name no)
@@
 			(project "Swadge-HW"
 				(path "/770c762f-3a30-4864-b7da-de353459cdd6/50e190c4-5ab4-41d8-900d-31bbecb31a92"
-					(reference "C16")
-					(unit 1)
-				)
+					(reference "C91")
+					(unit 1)
+				)

Commit message: Starting PCB
Very Rough Initial Layout
Parts:
- renumbered D10 to D91, L3 to L91
Changed lines of the file:
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@@
 		(in_pos_files yes)
 		(dnp no)
-		(property "Reference" "D10"
+		(property "Reference" "D91"
 			(at 103.632 120.65 90)
 			(show_name no)
@@
 			(project "Swadge-HW"
 				(path "/770c762f-3a30-4864-b7da-de353459cdd6/50e190c4-5ab4-41d8-900d-31bbecb31a92"
-					(reference "D10")
+					(reference "D91")
 					(unit 1)
 				)
@@
 		(in_pos_files yes)
 		(dnp no)
-		(property "Reference" "L3"
+		(property "Reference" "L91"
 			(at 110.49 113.03 90)
 			(show_name no)
@@
 			(project "Swadge-HW"
 				(path "/770c762f-3a30-4864-b7da-de353459cdd6/50e190c4-5ab4-41d8-900d-31bbecb31a92"
-					(reference "L3")
-					(unit 1)
-				)
+					(reference "L91")
+					(unit 1)
+				)

Commit message: major routing changes
Routed SPI
Started Test Routing Touch Inputs
Rough routing for LCD Power
Parts:
- C91, C93, C94: Cost @ 2.5k 0.0015 -> 0.0182
- C92, C95: Cost @ 2.5k 0.0035 -> 0.0121
- C96: Cost @ 2.5k 0.0079 -> 0.0198; LCSC C59461 -> C159801
- R91, R92: Cost @ 2.5k 0.0007 -> 0.0037
Changed lines of the file:
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@@
 			)
 		)
-		(property "Cost @ 2.5k" "0.0015"
+		(property "Cost @ 2.5k" "0.0182"
 			(at 238.76 107.95 0)
 			(hide yes)
@@
 			)
 		)
-		(property "Cost @ 2.5k" "0.0007"
+		(property "Cost @ 2.5k" "0.0037"
 			(at 177.8 124.46 0)
 			(hide yes)
@@
 			)
 		)
-		(property "Cost @ 2.5k" "0.0035"
+		(property "Cost @ 2.5k" "0.0121"
 			(at 78.74 120.65 0)
 			(hide yes)
@@
 			)
 		)
-		(property "Cost @ 2.5k" "0.0015"
+		(property "Cost @ 2.5k" "0.0182"
 			(at 246.38 107.95 0)
 			(hide yes)
@@
 			)
 		)
-		(property "Cost @ 2.5k" "0.0035"
+		(property "Cost @ 2.5k" "0.0121"
 			(at 116.84 41.91 0)
 			(hide yes)
@@
 			)
 		)
-		(property "Cost @ 2.5k" "0.0007"
+		(property "Cost @ 2.5k" "0.0037"
 			(at 86.36 102.87 0)
 			(hide yes)
@@
 			)
 		)
-		(property "LCSC" "C59461"
+		(property "LCSC" "C159801"
 			(at 119.38 120.65 0)
 			(hide yes)
@@
 			)
 		)
-		(property "Cost @ 2.5k" "0.0079"
+		(property "Cost @ 2.5k" "0.0198"
 			(at 119.38 120.65 0)
 			(hide yes)
@@
 			)
 		)
-		(property "Cost @ 2.5k" "0.0015"
+		(property "Cost @ 2.5k" "0.0182"
 			(at 83.82 41.91 0)
 			(hide yes)

Commit message: Restart Routing From Scratch
Total Restart of rough Routing with S3
Connections:
- net TFT_FMARK: no longer names the net of P2.11 (FMARK)
- no-connect marks 0 -> 1
Changed lines of the file:
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@@
 		(color 0 0 0 0)
+	)
+	(no_connect
+		(at 210.82 111.76)
 	)
 	(bus_entry
@@
 	(wire
 		(pts
-			(xy 210.82 111.76) (xy 209.55 111.76)
-		)
-		(stroke
-			(width 0)
-			(type default)
-		)
-	)
-	(wire
-		(pts
 			(xy 119.38 111.76) (xy 185.42 111.76)
 		)
@@
 		)
 	)
-	(global_label "TFT_FMARK"
-		(shape input)
-		(at 209.55 111.76 180)
-		(fields_autoplaced yes)
-		(effects
-			(font
-				(size 1.27 1.27)
-			)
-			(justify right)
-		)
-		(property "Intersheetrefs" "${INTERSHEET_REFS}"
-			(at 196.9769 111.6806 0)
-			(hide yes)
-			(show_name no)
-			(do_not_autoplace no)
-			(effects
-				(font
-					(size 1.27 1.27)
-				)
-				(justify right)
-			)
-		)
-	)
